File: Electronics/GrblPiB+-Industrial/GrblPi B+Industrial.brd (EAGLE design)
At the start: 156.1 x 98.8 mm, 82 parts, among them IC2 ATMEGA168-20P, K1 PIN20X2, SW2 SPST_TACT-EVQQ2, U1 EEPROM24

Commit message: Industrial Version:   Gerbers as ordered
Routing:
- net 5V: track 381.8 -> 447.7 mm
- net GPIO11: track 76.8 -> 75.0 mm
- net COOLANTENABLE: track 120.6 -> 119.9 mm
- net SDA1: track 86.7 -> 87.3 mm
- net GND: vias 8 -> 9
Other:
- board text added: "HITEMP.CO.ZA"
